File: kicad_files/kintsugi_v2.kicad_pcb (KiCad board)
At the start: 2 copper layers, 374.9 x 101.5 mm, 164 parts, among them J1 Conn_01x04, J2 Conn_01x04, J3 AudioJack4, J4 AudioJack4, SW1 RotaryEncoder_Switch, SW2 SW_Push, U1 ProMicro, U2 MCP23017_SP

Commit message: Finished routing on both sides. DRC and fillets pending.
Parts:
- J2: moved to F.Cu
- moved U2 0.13 mm to (34.9, 63.6)
- moved C1 0.13 mm to (27.3, 99.4), turned to 180 degrees
- moved C2 0.13 mm to (34.9, 99.4), turned to 0 degrees
- moved J2 0.13 mm to (27.3, 60.1), turned to 90 degrees
- moved R1 0.13 mm to (31.1, 99.4)
Routing:
- net VDD: track 0.00 -> 272.9 mm, vias 0 -> 1
- net SCL1: track 0.00 -> 251.0 mm, vias 0 -> 1
- net SDA1: track 0.00 -> 247.8 mm
- net COL9: track 122.3 -> 356.3 mm, vias 5 -> 9
- net COL10: track 125.9 -> 285.3 mm, vias 5 -> 11
- net COL11: track 130.2 -> 269.6 mm, vias 5 -> 11
- net COL13: track 123.1 -> 242.0 mm, vias 5 -> 7
- net COL14: track 126.7 -> 236.8 mm
- net COL12: track 88.0 -> 192.8 mm, vias 4 -> 6
- net COL8: track 288.7 -> 381.4 mm, vias 5 -> 7
- net ROW7: track 139.6 -> 218.0 mm, vias 0 -> 2
- net ROW10: track 160.3 -> 236.9 mm
- net COL15: track 129.8 -> 201.9 mm, vias 7 -> 8
- net ROW9: track 157.9 -> 227.5 mm, vias 0 -> 2
- net VSS: track 0.00 -> 63.2 mm
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